Commit message: for slam

File: src/mybot_description/urdf/mybot.xacro (robot description, xacro)
@@ -146,5 +146,5 @@
   <joint name="hokuyo_joint" type="fixed">
     <axis xyz="0 1 0" />
-    <origin xyz=".15 0 .1" rpy="0 0 0"/>
+    <origin xyz=".15 0 .15" rpy="0 0 0"/>
     <parent link="chassis"/>
     <child link="hokuyo"/>

Commit message: added aruco marker to gazebo and aruco detector

File: src/mybot_description/urdf/mybot.xacro (robot description, xacro)
@@ -140,5 +140,5 @@
   <joint name="camera_joint" type="fixed">
     <axis xyz="0 1 0" />
-    <origin xyz=".2 0 0" rpy="0 0 0"/>
+    <origin xyz=".2 0 0.5" rpy="0 0.15 0"/>
     <parent link="chassis"/>
     <child link="camera"/>

Commit message: aruco lesson

File: src/mybot_description/urdf/mybot.xacro (robot description, xacro)
@@ -140,7 +140,15 @@
   <joint name="camera_joint" type="fixed">
     <axis xyz="0 1 0" />
-    <origin xyz=".2 0 0.5" rpy="0 0.15 0"/>
+    <origin xyz=".2 0 0.5" rpy="0 0.1 0"/>
     <parent link="chassis"/>
     <child link="camera"/>
+  </joint>
+  <link name="camera_optical">
+    </link>
+  <joint name="camera_optical_joint" type="fixed">
+    <axis xyz="0 1 0" />
+    <origin xyz="0 0 0" rpy="-1.57 0 -1.57"/>
+    <parent link="camera"/>
+    <child link="camera_optical"/>
   </joint>
   <joint name="hokuyo_joint" type="fixed">

Commit message: problems with pointcloud in global cstmp

File: src/mybot_description/urdf/mybot.xacro (robot description, xacro)
@@ -158,4 +158,46 @@
     <child link="hokuyo"/>
   </joint>
+  <link name="depth_camera">
+      <collision>
+      <origin xyz="0 0 0" rpy="0 0 0"/>
+      <geometry>
+        <box size="${cameraSize} ${cameraSize} ${cameraSize}"/>
+      </geometry>
+    </collision>
+    <visual>
+      <origin xyz="0 0 0" rpy="0 0 0"/>
+      <geometry>
+        <box size="${cameraSize} ${cameraSize} ${cameraSize}"/>
+      </geometry>
+      <material name="blue"/>
+      <collision>
+      <origin xyz="0 0 0" rpy="0 0 0"/>
+      <geometry>
+        <box size="${cameraSize} ${cameraSize} ${cameraSize}"/>
+      </geometry>
+    </collision>
+    <visual>
+      <origin xyz="0 0 0" rpy="0 0 0"/>
+      <geometry>
+        <box size="${cameraSize} ${cameraSize} ${cameraSize}"/>
+      </geometry>
+      <material name="blue"/>
+    </visual>
+    </visual>
+  </link>
+  <joint name="depth_camera_joint" type="fixed">
+    <axis xyz="0 1 0" />
+    <origin xyz=".2 0 0" rpy="0 0 0"/>
+    <parent link="chassis"/>
+    <child link="depth_camera"/>
+  </joint>
+  <link name="depth_camera_optical">
+  </link>
+  <joint name="depth_camera_optical_joint" type="fixed">
+    <axis xyz="0 1 0" />
+    <origin xyz="0 0 0" rpy="-1.57 0 -1.57"/>
+    <parent link="depth_camera"/>
+    <child link="depth_camera_optical"/>
+  </joint>
   <!-- Hokuyo Laser -->
   <link name="hokuyo">

Commit message: base_link added

File: src/mybot_description/urdf/mybot.xacro (robot description, xacro)
@@ -6,4 +6,12 @@
   <xacro:include filename="$(find mybot_description)/urdf/materials.xacro" />
   <xacro:include filename="$(find mybot_description)/urdf/macros.xacro" />
+  <link name='base_link'>
+    </link>
+    <joint name="base_link_joint" type="fixed">
+    <axis xyz="0 1 0" />
+    <origin xyz="0 0 0.1" rpy="0 0 0"/>
+    <parent link="base_link"/>
+    <child link="chassis"/>
+  </joint>
   <link name='chassis'>
     <pose>0 0 0.1 0 0 0</pose>

Commit message: depth lesson ready

File: src/mybot_description/urdf/mybot.xacro (robot description, xacro)
@@ -10,5 +10,5 @@
     <joint name="base_link_joint" type="fixed">
     <axis xyz="0 1 0" />
-    <origin xyz="0 0 0.1" rpy="0 0 0"/>
+    <origin xyz="-0.1 0 0.1" rpy="0 0 0"/>
     <parent link="base_link"/>
     <child link="chassis"/>

Commit message: add new level

File: src/mybot_description/urdf/mybot.xacro (robot description, xacro)
@@ -196,5 +196,5 @@
   <joint name="depth_camera_joint" type="fixed">
     <axis xyz="0 1 0" />
-    <origin xyz=".2 0 0" rpy="0 0 0"/>
+    <origin xyz="0.2 0 0.3" rpy="-1.57 0.5 0"/>
     <parent link="chassis"/>
     <child link="depth_camera"/>
